File: PCB/Redwood.kicad_pcb (KiCad board)
At the start: 2 copper layers, 90 parts, among them SW1 SW_Push, SW10 SW_Push, SW11 SW_Push, SW12 SW_Push, SW13 SW_Push, SW14 SW_Push, SW15 SW_Push, SW16 SW_Push, SW17 SW_Push, SW18 SW_Push, SW19 SW_Push, SW2 SW_Push, SW20 SW_Push, SW21 SW_Push, SW22 SW_Push, SW23 SW_Push, SW24 SW_Push, SW25 SW_Push, SW26 SW_Push, SW27 SW_Push, SW28 SW_Push, SW29 SW_Push, SW3 SW_Push, SW30 SW_Push, SW31 SW_Push, SW32 SW_Push, SW33 SW_Push, SW34 SW_Push, SW35 SW_Push, SW36 SW_Push, SW37 SW_Push, SW38 SW_Push, SW39 SW_Push, SW4 SW_Push, SW40 SW_Push, SW41 SW_Push, SW42 SW_Push, SW43 SW_Push, SW44 SW_Push, SW47 EC11Ex, SW48 EC11Ex, SW5 SW_Push, SW6 SW_Push, SW7 SW_Push, SW8 SW_Push, SW9 SW_Push, U1 STM32F072C8Tx, U2 XC6206PxxxMR

Commit message: lot of pcb layouts, schematic mostly done
Parts:
- added C1: 100nF, Capacitor_SMD:C_0402_1005Metric, B.Cu at (187.6, 88.5)
- added C2: 100nF, Capacitor_SMD:C_0402_1005Metric, B.Cu at (187.6, 90.5)
- added C3: 100nF, Capacitor_SMD:C_0402_1005Metric, B.Cu at (187.6, 92.5)
- added C4: 100nF, Capacitor_SMD:C_0402_1005Metric, B.Cu at (187.6, 94.4)
- added C5: 100nF, Capacitor_SMD:C_0402_1005Metric, B.Cu at (187.6, 96.4)
- added C6: 1uF, Capacitor_SMD:C_0402_1005Metric, B.Cu at (161.9, 148.9)
- added C7: 1uF, Capacitor_SMD:C_0402_1005Metric, B.Cu at (169.9, 148.7)
- added C8: 100nF, Capacitor_SMD:C_0402_1005Metric, B.Cu at (232.6, 93.7)
- added J1: Conn_01x04_MountingPin, acheron_Connectors:MOLEX_781710004_MountingReliefs, B.Cu at (157.2, 138.1)
- added J2: Conn_01x16, acheron_Connectors:XFCN_F1004-H-16-20G-R_P1.0mm_MountingReliefs, F.Cu at (78.2, 131.8)
- added J3: Conn_01x16, acheron_Connectors:XFCN_F1004-H-16-20G-R_P1.0mm_MountingReliefs, F.Cu at (90.1, 131.8)
- added R1: 10k, Resistor_SMD:R_0402_1005Metric, B.Cu at (209.3, 83.3)
- added SW1: RST, Button_Switch_SMD:SW_SPST_SKQG_WithoutStem, B.Cu at (216.7, 84.9)
- added SW2: RST, Button_Switch_SMD:SW_SPST_SKQG_WithoutStem, B.Cu at (232.6, 88.1)
- D1, D10, D11, D12, D13, D14, D15, D16, D17, D18, D19, D2, D20, D21, D22, D23, D24, D25, D26, D27, D28, D29, D3, D30, D31, D32, D33, D34, D35, D36, D37, D38, D39, D4, D40, D41, D42, D5, D6, D7, D8, D9: moved to B.Cu
- U1: renamed from U2; moved to B.Cu
- U2: renamed from U1; moved to B.Cu
- moved D24 132.4 mm to (262.7, 42.1), turned to 90 degrees
- moved D23 127.9 mm to (259.6, 42.1), turned to 90 degrees
- moved D7 117.8 mm to (39.7, 67.5), turned to 90 degrees
- moved D1 117.0 mm to (39.7, 48.4), turned to 90 degrees
- moved D13 112.9 mm to (39.7, 86.5), turned to 90 degrees
- moved D36 112.9 mm to (262.7, 80.2), turned to 90 degrees
- moved D22 112.3 mm to (242.1, 41.3), turned to 90 degrees
- moved D30 112.1 mm to (262.7, 61.1), turned to 90 degrees
- moved D35 108.5 mm to (259.6, 80.2), turned to 90 degrees
- moved D29 107.8 mm to (259.6, 61.1), turned to 90 degrees
- moved D8 105.7 mm to (58.7, 63.5), turned to 90 degrees
- moved D2 104.7 mm to (58.7, 44.5), turned to 90 degrees
- moved D27 99.5 mm to (223.0, 57.1), turned to 90 degrees
- moved D21 98.3 mm to (223.0, 38.1), turned to 90 degrees
- moved D14 96.8 mm to (58.7, 82.5), turned to 90 degrees
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- renumbered SW6 to SW10, SW7 to SW11, SW8 to SW12, SW9 to SW13, SW10 to SW14, SW11 to SW15, SW12 to SW16, SW13 to SW17, SW14 to SW18, SW15 to SW19, SW16 to SW20, SW17 to SW21, SW18 to SW22, SW19 to SW23, SW20 to SW24, SW21 to SW25, SW22 to SW26, SW23 to SW27, SW24 to SW28, SW25 to SW29, SW47 to SW3, SW26 to SW30, SW27 to SW31, SW28 to SW32, SW29 to SW33, SW30 to SW34, SW31 to SW35, SW32 to SW36, SW33 to SW37, SW34 to SW38, SW35 to SW39, SW48 to SW4, SW36 to SW40, SW37 to SW41, SW38 to SW45, SW39 to SW46, SW40 to SW47, SW41 to SW48, SW1 to SW5, SW2 to SW6, SW3 to SW7, SW4 to SW8, SW5 to SW9
Connections:
- U2 pad 11: unconnected-(U1-PA1-Pad11) -> COL0
- U2 pad 12: unconnected-(U1-PA2-Pad12) -> COL1
- U2 pad 13: unconnected-(U1-PA3-Pad13) -> ROW5
- U2 pad 14: unconnected-(U1-PA4-Pad14) -> ROW4
- U2 pad 15: unconnected-(U1-PA5-Pad15) -> ROW3
- U2 pad 16: unconnected-(U1-PA6-Pad16) -> COL2
- U2 pad 2: unconnected-(U1-PC13-Pad2) -> ROW2
- U2 pad 25: unconnected-(U1-PB12-Pad25) -> COL3
- U2 pad 26: unconnected-(U1-PB13-Pad26) -> COL4
- U2 pad 27: unconnected-(U1-PB14-Pad27) -> COL5
- U2 pad 28: unconnected-(U1-PB15-Pad28) -> ROW6
- U2 pad 3: unconnected-(U1-PC14-Pad3) -> ROW1
- U2 pad 4: unconnected-(U1-PC15-Pad4) -> ROW0
Routing:
- net COL5: track 0.00 -> 85.7 mm
- net COL0: track 0.00 -> 85.7 mm
- net COL4: track 0.00 -> 76.2 mm
- net COL1: track 0.00 -> 76.2 mm
- net COL3: track 0.00 -> 76.2 mm
- net COL2: track 0.00 -> 76.2 mm
- net Net-(D42-A): track 0.00 -> 9.52 mm
- net Net-(D37-A): track 0.00 -> 9.52 mm
Other:
- board outline added: 15.9 x 54 mm

Commit message: proto pcb ordered
Parts:
- added H1: MountingHole, acheron_Hardware:MouseBite_IPC7351, F.Cu at (138.0, 111.8)
- added H2: MountingHole, acheron_Hardware:MouseBite_IPC7351, F.Cu at (135.0, 111.5)
- added H3: MountingHole, acheron_Hardware:MouseBite_IPC7351, F.Cu at (138.0, 49.5)
- added H4: MountingHole, acheron_Hardware:MouseBite_IPC7351, F.Cu at (135.0, 49.5)
- added H5: MountingHole, acheron_Hardware:MouseBite_IPC7351, F.Cu at (138.0, 78.5)
- added H6: MountingHole, acheron_Hardware:MouseBite_IPC7351, F.Cu at (135.0, 78.5)
- D1, D10, D11, D12, D13, D14, D15, D16, D17, D18, D19, D2, D20, D21, D22, D23, D24, D25, D26, D28, D29, D3, D30, D31, D32, D33, D34, D35, D36, D37, D38, D39, D4, D40, D41, D42, D5, D6, D7, D8, D9: footprint acheron_Components:D_SOD-123 -> Diode_SMD:D_SOD-123
- D27: value D_Small -> 1N4148; footprint acheron_Components:D_SOD-123 -> Diode_SMD:D_SOD-123
- J2, J3: moved to B.Cu
- SW1: value RST -> BOOT
- SW2: value RST -> RESET
- moved C8 107.7 mm to (126.2, 76.3), turned to -100 degrees
- moved C6 107.7 mm to (111.1, 54.0), turned to -10 degrees
- moved C7 107.6 mm to (109.6, 59.6), turned to -10 degrees
- moved U1 107.2 mm to (110.1, 56.7), turned to 80 degrees
- moved SW2 103.4 mm to (130.4, 72.1), turned to -90 degrees
- moved U2 98.7 mm to (104.9, 68.7), turned to 80 degrees
- moved J1 94.9 mm to (117.7, 51.9), turned to 180 degrees
- moved C2 91.6 mm to (99.5, 65.3), turned to -100 degrees
- moved SW1 89.2 mm to (130.4, 62.5), turned to 90 degrees
- moved C4 86.6 mm to (103.3, 74.8), turned to -10 degrees
- moved C5 85.6 mm to (108.7, 63.4), turned to 170 degrees
- moved R1 84.5 mm to (126.4, 66.5), turned to 80 degrees
- moved C3 81.9 mm to (107.5, 75.6), turned to -10 degrees
- moved C1 79.1 mm to (110.0, 73.4), turned to -100 degrees
- moved J2 78.0 mm to (145.8, 92.9)
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Connections:
- C1 pad 1: +3V3 -> +3.3V
- C2 pad 1: +3V3 -> +3.3V
- C3 pad 1: +3V3 -> +3.3V
- C4 pad 1: +3V3 -> +3.3V
- C5 pad 1: +3V3 -> +3.3V
- J2 pad 10: ROW0 -> ROW3
- J2 pad 8: ROW2 -> ROW5
- J2 pad 9: ROW1 -> ROW4
- J2 pad MP: (no net) -> GND
- J3 pad 7: ROW0 -> ROW3
- J3 pad 8: ROW1 -> ROW4
- J3 pad 9: ROW2 -> ROW5
- J3 pad MP: (no net) -> GND
- U2 pad 10: unconnected-(U2-PA0-Pad10) -> COL2
- U2 pad 11: COL0 -> COL3
- U2 pad 12: COL1 -> COL4
- U2 pad 13: ROW5 -> unconnected-(U2-PA3-Pad13)
- U2 pad 14: ROW4 -> unconnected-(U2-PA4-Pad14)
- U2 pad 15: ROW3 -> unconnected-(U2-PA5-Pad15)
- U2 pad 16: COL2 -> ROW2
- U2 pad 17: unconnected-(U2-PA7-Pad17) -> ROW1
- U2 pad 2: ROW2 -> ENCODER_B
- U2 pad 25: COL3 -> unconnected-(U2-PB12-Pad25)
- U2 pad 26: COL4 -> unconnected-(U2-PB13-Pad26)
- U2 pad 27: COL5 -> unconnected-(U2-PB14-Pad27)
- U2 pad 28: ROW6 -> unconnected-(U2-PB15-Pad28)
- U2 pad 29: unconnected-(U2-PA8-Pad29) -> ROW0
- U2 pad 3: ROW1 -> ENCODER_A
- U2 pad 37: ENCODER_B -> unconnected-(U2-PA14-Pad37)
- U2 pad 38: ENCODER_A -> unconnected-(U2-PA15-Pad38)
- U2 pad 4: ROW0 -> COL0
- U2 pad 41: unconnected-(U2-PB5-Pad41) -> ROW3
- U2 pad 42: unconnected-(U2-PB6-Pad42) -> ROW4
- U2 pad 43: unconnected-(U2-PB7-Pad43) -> ROW5
- U2 pad 45: unconnected-(U2-PB8-Pad45) -> ROW6
- U2 pad 46: unconnected-(U2-PB9-Pad46) -> COL5
- U2 pad 5: unconnected-(U2-PF0-Pad5) -> COL1
Routing:
- net ENCODER_A: track 0.00 -> 214.4 mm, vias 0 -> 1
- net ENCODER_B: track 0.00 -> 202.6 mm, vias 0 -> 1
- net ROW3: track 0.00 -> 191.8 mm, vias 0 -> 4
- net COL3: track 76.2 -> 256.0 mm, vias 0 -> 3
- net COL4: track 76.2 -> 255.7 mm, vias 0 -> 4
- net COL2: track 76.2 -> 254.5 mm, vias 0 -> 3
- net COL0: track 85.7 -> 260.6 mm, vias 0 -> 3
- net COL1: track 76.2 -> 250.3 mm, vias 0 -> 4
- net ROW4: track 0.00 -> 172.9 mm, vias 0 -> 4
- net ROW6: track 0.00 -> 164.9 mm, vias 0 -> 2
- net COL5: track 85.7 -> 244.2 mm, vias 0 -> 3
- net ROW5: track 0.00 -> 156.0 mm, vias 0 -> 2
- net ROW1: track 0.00 -> 118.4 mm, vias 0 -> 2
- net ROW2: track 0.00 -> 117.8 mm, vias 0 -> 2
- net ROW0: track 0.00 -> 107.8 mm
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- added copper zone on B.Cu, net GND
- added copper zone on F.Cu, net GND
Other:
- board size 15.9 x 54 mm -> 255.4 x 94.7 mm
