File: PCB/Matrix.kicad_sch (KiCad schematic)
At the start: 86 parts, among them SW1 SW_Push, SW10 SW_Push, SW11 SW_Push, SW12 SW_Push, SW13 SW_Push, SW14 SW_Push, SW15 SW_Push, SW16 SW_Push, SW17 SW_Push, SW18 SW_Push, SW19 SW_Push, SW2 SW_Push, SW20 SW_Push, SW21 SW_Push, SW22 SW_Push, SW23 SW_Push, SW24 SW_Push, SW25 SW_Push, SW26 SW_Push, SW27 SW_Push, SW28 SW_Push, SW29 SW_Push, SW3 SW_Push, SW30 SW_Push, SW31 SW_Push, SW32 SW_Push, SW33 SW_Push, SW34 SW_Push, SW35 SW_Push, SW36 SW_Push, SW37 SW_Push, SW38 SW_Push, SW39 SW_Push, SW4 SW_Push, SW40 SW_Push, SW41 SW_Push, SW42 SW_Push, SW43 SW_Push, SW44 SW_Push, SW5 SW_Push, SW6 SW_Push, SW7 SW_Push, SW8 SW_Push, SW9 SW_Push

Commit message: lot of pcb layouts, schematic mostly done
Parts:
- renumbered SW6 to SW10, SW7 to SW11, SW8 to SW12, SW9 to SW13, SW10 to SW14, SW11 to SW15, SW12 to SW16, SW13 to SW17, SW14 to SW18, SW15 to SW19, SW16 to SW20, SW17 to SW21, SW18 to SW22, SW19 to SW23, SW20 to SW24, SW21 to SW25, SW22 to SW26, SW23 to SW27, SW24 to SW28, SW25 to SW29, SW26 to SW30, SW27 to SW31, SW28 to SW32, SW29 to SW33, SW30 to SW34, SW31 to SW35, SW32 to SW36, SW33 to SW37, SW34 to SW38, SW35 to SW39, SW36 to SW40, SW37 to SW41, SW38 to SW45, SW39 to SW46, SW40 to SW47, SW41 to SW48, SW1 to SW5, SW2 to SW6, SW3 to SW7, SW4 to SW8, SW5 to SW9

Commit message: proto pcb ordered
Parts:
- D1, D10, D11, D12, D13, D14, D15, D16, D17, D18, D19, D2, D20, D21, D22, D23, D24, D25, D26, D28, D29, D3, D30, D31, D32, D33, D34, D35, D36, D37, D38, D39, D4, D40, D41, D42, D5, D6, D7, D8, D9: footprint acheron_Components:D_SOD-123 -> Diode_SMD:D_SOD-123
- D27: value D_Small -> 1N4148; footprint acheron_Components:D_SOD-123 -> Diode_SMD:D_SOD-123
