File: PCB/Redwood.kicad_sch (KiCad schematic)
At the start: 21 parts, among them J1 Conn_01x04_MountingPin, SW45 RST, SW46 RST, SW47 EC11Ex, SW48 EC11Ex, U1 STM32F072C8Tx, U2 XC6206PxxxMR

Commit message: lot of pcb layouts, schematic mostly done
Parts:
- removed C1: 4.7uF, symbol Device:C
- removed C10, C11, C12, C13: 100nF, symbol Device:C
- added J2, J3: Conn_01x16, acheron_Connectors:XFCN_F1004-H-16-20G-R_P1.0mm_MountingReliefs, symbol Connector_Generic:Conn_01x16
- C1: renamed from C2; footprint (none) -> Capacitor_SMD:C_0402_1005Metric
- C2: renamed from C3; footprint (none) -> Capacitor_SMD:C_0402_1005Metric
- C3: renamed from C4; footprint (none) -> Capacitor_SMD:C_0402_1005Metric
- C4: renamed from C5; footprint (none) -> Capacitor_SMD:C_0402_1005Metric
- C5: renamed from C6; footprint (none) -> Capacitor_SMD:C_0402_1005Metric
- C6: renamed from C7; footprint (none) -> Capacitor_SMD:C_0402_1005Metric
- C7: renamed from C8; footprint (none) -> Capacitor_SMD:C_0402_1005Metric
- C8: renamed from C9; footprint (none) -> Capacitor_SMD:C_0402_1005Metric
- J1: footprint (none) -> acheron_Connectors:MOLEX_781710004_MountingReliefs
- R1: footprint (none) -> Resistor_SMD:R_0402_1005Metric
- SW1: renamed from SW45; footprint (none) -> Button_Switch_SMD:SW_SPST_SKQG_WithoutStem
- SW2: renamed from SW46; footprint (none) -> Button_Switch_SMD:SW_SPST_SKQG_WithoutStem
- renumbered SW47 to SW3, SW48 to SW4, U2 to U1, U1 to U2
Connections:
- net +5V: now also J2.2 (Pin_2), J3.15 (Pin_15)
- net ENCODER_A: now also J2.6 (Pin_6), J3.11 (Pin_11)
- net ENCODER_B: now also J2.5 (Pin_5), J3.12 (Pin_12)
- net GND: now also J2.1 (Pin_1), J3.16 (Pin_16)
- net COL0: now reaches U2.11 (PA1)
- net COL0: now also J2.16 (Pin_16), J3.1 (Pin_1)
- net COL1: now reaches U2.12 (PA2)
- net COL1: now also J2.15 (Pin_15), J3.2 (Pin_2)
- net ROW5: now reaches U2.13 (PA3)
- net ROW4: now reaches U2.14 (PA4)
- net ROW3: now reaches U2.15 (PA5)
- net COL2: now reaches U2.16 (PA6)
- net COL2: now also J2.14 (Pin_14), J3.3 (Pin_3)
- net ROW2: now reaches U2.2 (PC13)
- net ROW2: now also J2.8 (Pin_8), J3.9 (Pin_9)
- net COL3: now reaches U2.25 (PB12)
- net COL3: now also J2.13 (Pin_13), J3.4 (Pin_4)
- net COL4: now reaches U2.26 (PB13)
- net COL4: now also J2.12 (Pin_12), J3.5 (Pin_5)
- net COL5: now reaches U2.27 (PB14)
- net COL5: now also J2.11 (Pin_11), J3.6 (Pin_6)
- net ROW6: now reaches U2.28 (PB15)
- net ROW6: now also J2.7 (Pin_7), J3.10 (Pin_10)
- net ROW1: now reaches U2.3 (PC14)
- net ROW1: now also J2.9 (Pin_9), J3.8 (Pin_8)
- net ROW0: now reaches U2.4 (PC15)
- net ROW0: now also J2.10 (Pin_10), J3.7 (Pin_7)
- new net RGB_LED: J2.4 (Pin_4), J3.13 (Pin_13)
Other:
- moved on the sheet: C1, C2, C3, C4, C5, SW3, SW4

Commit message: proto pcb ordered
Parts:
- added H1, H2, H3, H4, H5, H6: MountingHole, acheron_Hardware:MouseBite_IPC7351, symbol Mechanical:MountingHole
- J2, J3: symbol Connector_Generic:Conn_01x16 -> Connector_Generic_MountingPin:Conn_01x16_MountingPin
- SW1: value RST -> BOOT
- SW2: value RST -> RESET
Connections:
- net +3V3 is gone; now on net +3.3V: C1.1, C2.1, C3.1, C4.1, C5.1
- net COL0: now also U2.4 (PC15); no longer U2.11 (PA1)
- net COL1: now also U2.5 (PF0); no longer U2.12 (PA2)
- net COL2: now also U2.10 (PA0); no longer U2.16 (PA6)
- net COL3: now also U2.11 (PA1); no longer U2.25 (PB12)
- net COL4: now also U2.12 (PA2); no longer U2.26 (PB13)
- net COL5: now also U2.46 (PB9); no longer U2.27 (PB14)
- net ENCODER_A: now also U2.3 (PC14); no longer U2.38 (PA15)
- net ENCODER_B: now also U2.2 (PC13); no longer U2.37 (PA14)
- net GND: now also J2.MP (MountPin), J3.MP (MountPin)
- net ROW0: now also U2.29 (PA8); no longer J2.10 (Pin_10), J3.7 (Pin_7), U2.4 (PC15)
- net ROW1: now also U2.17 (PA7); no longer J2.9 (Pin_9), J3.8 (Pin_8), U2.3 (PC14)
- net ROW2: now also U2.16 (PA6); no longer J2.8 (Pin_8), J3.9 (Pin_9), U2.2 (PC13)
- net ROW3: now also J2.10 (Pin_10), J3.7 (Pin_7), U2.41 (PB5); no longer U2.15 (PA5)
- net ROW4: now also J2.9 (Pin_9), J3.8 (Pin_8), U2.42 (PB6); no longer U2.14 (PA4)
- net ROW5: now also J2.8 (Pin_8), J3.9 (Pin_9), U2.43 (PB7); no longer U2.13 (PA3)
- net ROW6: now also U2.45 (PB8); no longer U2.28 (PB15)

Commit message: v2
Connections:
- net +5V: no longer J2.2 (Pin_2), J3.15 (Pin_15)
- net COL0: now also J2.11 (Pin_11), J3.6 (Pin_6); no longer J2.16 (Pin_16), J3.1 (Pin_1)
- net COL1: now also J2.12 (Pin_12), J3.5 (Pin_5); no longer J2.15 (Pin_15), J3.2 (Pin_2)
- net COL2: now also J2.13 (Pin_13), J3.4 (Pin_4); no longer J2.14 (Pin_14), J3.3 (Pin_3)
- net COL3: now also J2.14 (Pin_14), J3.3 (Pin_3); no longer J2.13 (Pin_13), J3.4 (Pin_4)
- net COL4: now also J2.15 (Pin_15), J3.2 (Pin_2); no longer J2.12 (Pin_12), J3.5 (Pin_5)
- net COL5: now also J2.16 (Pin_16), J3.1 (Pin_1); no longer J2.11 (Pin_11), J3.6 (Pin_6)
- net RGB_LED: no longer names the net of J2.4 (Pin_4)
- net RGB_LED: no longer J3.13 (Pin_13)
